File: pcb/tasty-totem-board/tasty-totem-board.kicad_sch (KiCad schematic)
At the start: 6 parts, among them J1 Motor Header, J2 IR Receive Header, J3 IR Send Header, J4 LED Strip Header, U1 ESP32-DEVKIT-V1, U2 L9110

Commit message: Checkpoint current version of PCB design files
Parts:
- added J5: Activation Switch, Connector_PinSocket_2.54mm:PinSocket_1x02_P2.54mm_Horizontal, symbol Connector:Conn_01x02_Socket
- added J6: AUX LED Strip, Connector_PinSocket_2.54mm:PinSocket_1x03_P2.54mm_Horizontal, symbol Connector:Conn_01x03_Socket
- added J7: Light Sensor, Connector_PinSocket_2.54mm:PinSocket_1x03_P2.54mm_Horizontal, symbol Connector:Conn_01x03_Socket
- added J8: Multi-use A, Connector_PinSocket_2.54mm:PinSocket_1x03_P2.54mm_Horizontal, symbol Connector:Conn_01x03_Socket
- J1: footprint (none) -> Connector_PinSocket_2.54mm:PinSocket_1x06_P2.54mm_Horizontal
- J2, J4: footprint (none) -> Connector_PinSocket_2.54mm:PinSocket_1x03_P2.54mm_Horizontal
- J3: footprint (none) -> Connector_PinSocket_2.54mm:PinSocket_1x02_P2.54mm_Horizontal
- U2: footprint (none) -> Package_DIP:DIP-8_W7.62mm
Connections:
- net +5V: now also J6.1 (Pin_1), J7.1 (Pin_1), J8.1 (Pin_1)
- net A PHASE OF C2 ENCODER: now also U1.4 (D2); no longer U1.14 (D22)
- net B PHASE OF C1 ENCODER: now also U1.3 (D15); no longer U1.15 (D23)
- net GND: now also J5.2 (Pin_2), J6.3 (Pin_3), J7.3 (Pin_3), J8.3 (Pin_3)
- net AUX Strip: now reaches U1.19 (D34)
- net AUX Strip: now also J6.2 (Pin_2)
- net LIGHT SENSOR: now reaches U1.21 (D32)
- net LIGHT SENSOR: now also J7.2 (Pin_2)
- net ACTIVATION SWITCH: now reaches U1.24 (D26)
- net ACTIVATION SWITCH: now also J5.1 (Pin_1)
- net SIGA: now reaches U1.28 (D13)
- net SIGA: now also J8.2 (Pin_2)
