File: pcb/7-segment-driver/7-segment-driver.kicad_sch (KiCad schematic)
At the start: 26 parts, among them J1 AVR-ISP-6, U1 74HC595, U2 74HC595, U3 ATtiny84A-SS, U4 SH18101AS, U6 SH18101AS

Commit message: Checkpoint PCB files.
Parts:
- R1, R2, R3: value R -> 120
Changed lines of the file:
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@@
 	(label "1.G"
 		(at 240.03 134.62 0)
+		(fields_autoplaced yes)
 		(effects
 			(font
@@
 	(label "1.D"
 		(at 240.03 119.38 0)
+		(fields_autoplaced yes)
 		(effects
 			(font
@@
 	(label "DI"
 		(at 60.96 166.37 0)
+		(fields_autoplaced yes)
 		(effects
 			(font
@@
 	(label "1.F"
 		(at 156.21 127 0)
+		(fields_autoplaced yes)
 		(effects
 			(font
@@
 	(label "10.C"
 		(at 156.21 64.77 0)
+		(fields_autoplaced yes)
 		(effects
 			(font
@@
 	(label "1.H"
 		(at 240.03 139.7 0)
+		(fields_autoplaced yes)
 		(effects
 			(font
@@
 	(label "10.G"
 		(at 156.21 74.93 0)
+		(fields_autoplaced yes)
 		(effects
 			(font
@@
 	(label "1.G"
 		(at 156.21 129.54 0)
+		(fields_autoplaced yes)
 		(effects
 			(font
@@
 	(label "rclk"
 		(at 135.89 127 0)
+		(fields_autoplaced yes)
 		(effects
 			(font
@@
 	(label "1.A"
 		(at 240.03 104.14 0)
+		(fields_autoplaced yes)
 		(effects
 			(font
@@
 	(label "1.A"
 		(at 156.21 114.3 0)
+		(fields_autoplaced yes)
 		(effects
 			(font
@@
 	(label "rclk"
 		(at 68.58 67.31 0)
+		(fields_autoplaced yes)
 		(effects
 			(font
@@
 	(label "CLK"
 		(at 68.58 69.85 0)
+		(fields_autoplaced yes)
 		(effects
 			(font
@@
 	(label "srclr"
 		(at 135.89 67.31 0)
+		(fields_autoplaced yes)
 		(effects
 			(font
@@
 	(label "1.B"
 		(at 240.03 109.22 0)
+		(fields_autoplaced yes)
 		(effects
 			(font
@@
 	(label "rclk"
 		(at 135.89 72.39 0)
+		(fields_autoplaced yes)
 		(effects
 			(font
@@
 	(label "10.F"
 		(at 156.21 72.39 0)
+		(fields_autoplaced yes)
 		(effects
 			(font
@@
 	(label "10.C"
 		(at 240.03 59.69 0)
+		(fields_autoplaced yes)
 		(effects
 			(font
@@
 	(label "DI"
 		(at 63.5 127 0)
+		(fields_autoplaced yes)
 		(effects
 			(font
@@
 	(label "10.D"
 		(at 240.03 64.77 0)
+		(fields_autoplaced yes)
 		(effects
 			(font
@@
 	(label "1.C"
 		(at 240.03 114.3 0)
+		(fields_autoplaced yes)
 		(effects
 			(font
@@
 	(label "10.B"
 		(at 156.21 62.23 0)
+		(fields_autoplaced yes)
 		(effects
 			(font
@@
 	(label "ser"
 		(at 135.89 59.69 0)
+		(fields_autoplaced yes)
 		(effects
 			(font
@@
 	(label "ser"
 		(at 68.58 59.69 0)
+		(fields_autoplaced yes)
 		(effects
 			(font
@@
 	(label "1.D"
 		(at 156.21 121.92 0)
+		(fields_autoplaced yes)
 		(effects
 			(font
@@
 	(label "srclk"
 		(at 135.89 64.77 0)
+		(fields_autoplaced yes)
 		(effects
 			(font
@@
 	(label "10.A"
 		(at 240.03 49.53 0)
+		(fields_autoplaced yes)
 		(effects
 			(font
@@
 	(label "1.C"
 		(at 156.21 119.38 0)
+		(fields_autoplaced yes)
 		(effects
 			(font
@@
 	(label "10.A"
 		(at 156.21 59.69 0)
+		(fields_autoplaced yes)
 		(effects
 			(font
@@
 	(label "srclr"
 		(at 135.89 121.92 0)
+		(fields_autoplaced yes)
 		(effects
 			(font
@@
 	(label "1.F"
 		(at 240.03 129.54 0)
+		(fields_autoplaced yes)
 		(effects
 			(font
@@
 	(label "10.H"
 		(at 156.21 77.47 0)
+		(fields_autoplaced yes)
 		(effects
 			(font
@@
 	(label "10.B"
 		(at 240.03 54.61 0)
+		(fields_autoplaced yes)
 		(effects
 			(font
@@
 	(label "DO"
 		(at 63.5 124.46 0)
+		(fields_autoplaced yes)
 		(effects
 			(font
@@
 	(label "oe"
 		(at 68.58 82.55 0)
+		(fields_autoplaced yes)
 		(effects
 			(font
@@
 	(label "1.H"
 		(at 156.21 132.08 0)
+		(fields_autoplaced yes)
 		(effects
 			(font
@@
 	(label "oe"
 		(at 135.89 129.54 0)
+		(fields_autoplaced yes)
 		(effects
 			(font
@@
 	(label "oe"
 		(at 135.89 74.93 0)
+		(fields_autoplaced yes)
 		(effects
 			(font
@@
 	(label "10.E"
 		(at 240.03 69.85 0)
+		(fields_autoplaced yes)
 		(effects
 			(font
@@
 	(label "10.H"
 		(at 240.03 85.09 0)
+		(fields_autoplaced yes)
 		(effects
 			(font
@@
 	(label "DO"
 		(at 68.58 72.39 0)
+		(fields_autoplaced yes)
 		(effects
 			(font
@@
 	(label "10.G"
 		(at 240.03 80.01 0)
+		(fields_autoplaced yes)
 		(effects
 			(font
@@
 	(label "DO"
 		(at 60.96 168.91 0)
+		(fields_autoplaced yes)
 		(effects
 			(font
@@
 	(label "10.E"
 		(at 156.21 69.85 0)
+		(fields_autoplaced yes)
 		(effects
 			(font
@@
 	(label "srclk"
 		(at 135.89 119.38 0)
+		(fields_autoplaced yes)
 		(effects
 			(font
@@
 	(label "EN"
 		(at 60.96 173.99 0)
+		(fields_autoplaced yes)
 		(effects
 			(font
@@
 	(label "1.E"
 		(at 240.03 124.46 0)
+		(fields_autoplaced yes)
 		(effects
 			(font
@@
 	(label "CLK"
 		(at 63.5 129.54 0)
+		(fields_autoplaced yes)
 		(effects
 			(font
@@
 	(label "EN"
 		(at 68.58 77.47 0)
+		(fields_autoplaced yes)
 		(effects
 			(font
@@
 	(label "1.B"
 		(at 156.21 116.84 0)
+		(fields_autoplaced yes)
 		(effects
 			(font
@@
 	(label "srclr"
 		(at 68.58 64.77 0)
+		(fields_autoplaced yes)
 		(effects
 			(font
@@
 	(label "1.E"
 		(at 156.21 124.46 0)
+		(fields_autoplaced yes)
 		(effects
 			(font
@@
 	(label "CLK"
 		(at 60.96 171.45 0)
+		(fields_autoplaced yes)
 		(effects
 			(font
@@
 	(label "DI"
 		(at 68.58 74.93 0)
+		(fields_autoplaced yes)
 		(effects
 			(font
@@
 	(label "10.D"
 		(at 156.21 67.31 0)
+		(fields_autoplaced yes)
 		(effects
 			(font
@@
 	(label "srclk"
 		(at 68.58 62.23 0)
+		(fields_autoplaced yes)
 		(effects
 			(font
@@
 	(label "10.F"
 		(at 240.03 74.93 0)
+		(fields_autoplaced yes)
 		(effects
 			(font
@@
 			)
 		)
-		(property "Value" "R"
+		(property "Value" "120"
 			(at 236.22 50.8 90)
 			(effects
@@
 			)
 		)
-		(property "Value" "R"
+		(property "Value" "120"
 			(at 236.22 61.214 90)
 			(effects
@@
 			)
 		)
-		(property "Value" "R"
+		(property "Value" "120"
 			(at 236.474 56.134 90)
 			(effects
