File: pcb/rotary-control/rotary-control.kicad_sch (KiCad schematic)
At the start: 12 parts, among them J1 input, J2 output, J3 power, J4 neopixel, J5 AVR_SPI_PRG_6PTH, J6 encoder

Commit message: Checkpoint PCB files.
Parts:
- removed J1: input, rotary-control:1X05, symbol rotary-control-eagle-import:CONN_05
- removed J2: output, rotary-control:1X05, symbol rotary-control-eagle-import:CONN_05
- removed J3: power, rotary-control:1X02, symbol rotary-control-eagle-import:CONN_02
- removed R1: 4K7, rotary-control:0805, symbol rotary-control-eagle-import:RESISTOR
- added H1, H2: MountingHole, MountingHole:MountingHole_2.7mm_M2.5_Pad, symbol Mechanical:MountingHole
- added J1: SPI-Comm, Garth:RJ11-Straight, symbol Garth Libraries:SPI-Comm-Jack
- C1: footprint rotary-control:1206 -> Capacitor_SMD:C_1206_3216Metric_Pad1.33x1.80mm_HandSolder
- J4: footprint rotary-control:1X03 -> Connector_PinHeader_2.54mm:PinHeader_1x03_P2.54mm_Vertical
- J6: footprint rotary-control:1X05 -> Connector_PinHeader_2.54mm:PinHeader_1x05_P2.54mm_Vertical
- U$2: footprint rotary-control:SO14 -> Package_SO:SOIC-14_3.9x8.7mm_P1.27mm
Connections:
- net CS: now also J1.5 (EN)
- net DI: now also J1.2 (DI)
- net DO: now also J1.3 (DO)
- net GND: now also J1.6 (GND)
- net SCLK: now also J1.4 (SCK)
- net VCC: now also J1.1 (VCC)
- no-connect marks 0 -> 3
Other:
- moved on the sheet: C2, C4, R8
